File: eagle/norns-shield-211028.brd (EAGLE design)
At the start: 85.1 x 80 mm, 80 parts, among them J1 TRS-IN, J2 TRS-OUT, J3 ISP-ROW, Q1 ASFL-12.288mhz, SW1 PVA1, SW2 PVA1, SW3 PVA1, U1 CS4270, X1 RASPI_BOARD_B+#_E3

Commit message: add all versions, draft
Parts:
- removed /INA, /INB, /LRCK, /MCLK, /OUTA, /OUTB, /RESET, /SCL, /SCLK, /SDA, /SDIN, /SDOUT: TPTP12R, testpad:TP12R
- removed J1: TRS-IN, lines:SJ-3523-SMT
- removed J2: TRS-OUT, lines:SJ-3523-SMT
- added C18, C47, C63: 100n, rcl:C0603
- added C19, C43: 10u, rcl:C0805
- added C20, C88: 10n, rcl:C0603
- added C21, C24, C27, C30: 22u, rcl:C1206
- added C22, C28: 1n5, rcl:C0603
- added C23, C29: 470p, rcl:C0603
- added C25: 2200p COG, rcl:C0603
- added C26: 6n8, rcl:C0603
- added IC1, IC2, IC4: TL072D, linear:SO08
- added J-IN, J-OUT: JACK-TRS-SW, lines:JACK4832.2330
- added L3: FERRITE, rc-master-smd:L0805
- added R16, R23: 2k32, rcl:R0603
- added R17, R24: 4k99, rcl:R0603
- added R19: 1k33, rcl:R0603
- added R20: 4k42, rcl:R0603
- added R21: 1k5, rcl:R0603
- added R22: 715, rcl:R0603
- added R25: 47k, rcl:R0603
- added R27, R30: 560, rcl:R0603
- added R5: 634, rcl:R0603
- added R6: 91, rcl:R0603
- added TP1, TP2: TPB1,27, testpad:B1,27
- added U11: TPS793, lines:SSOP6
- C11: value 220p COG -> 470p COG
- C12: value 10u -> 470p COG; device rcl:C0805 -> rcl:C0603
- C13: value 220p COG -> 2700p COG
- C14, C16: value 3.3u -> 10n; device rcl:C0805 -> rcl:C0603
- C15: value 2700p COG -> 2200p COG
- C17: value 2700p COG -> 6n8
- C4: value 100n -> 2700p COG
- R10: value 1.5k -> 634
- R11: value 10k -> 1k33
- R12: value 470 -> 4k42
- R13: value 10k -> 1k5
- R14: value 470 -> 715
- R18: value 0 -> 47k
- R7: value 3.3k -> 91
- R8: value 1.5k -> 10k
- R9: value 3.3k -> 10k
- U1: value CS4270 -> CS4271; device lines:TSSOP24 -> lines:SOP28
- moved C10 24.2 mm to (11.1, 45.1)
- moved C16 23.7 mm to (21.0, 26.0)
- moved R7 23.2 mm to (11.4, 38.7), turned to 180 degrees
- moved C11 23.1 mm to (11.4, 40.6), turned to 180 degrees
- moved C15 22.5 mm to (29.2, 27.9), turned to 180 degrees
- moved R8 22.0 mm to (11.4, 43.2), turned to 0 degrees
- moved R12 21.7 mm to (26.7, 30.2), turned to 270 degrees
- moved R11 21.7 mm to (24.8, 35.6), turned to 90 degrees
- moved C1 21.3 mm to (27.9, 7.62), turned to 0 degrees
- moved C2 20.8 mm to (27.9, 9.53), turned to 0 degrees
- moved C4 20.0 mm to (9.84, 36.8), turned to 0 degrees
- moved R15 18.5 mm to (22.2, 10.2), turned to 0 degrees
- moved C5 16.9 mm to (22.9, 46.4), turned to 180 degrees
- moved R18 16.5 mm to (35.6, 27.9), turned to 0 degrees
- moved R14 14.3 mm to (29.2, 34.3), turned to 180 degrees
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Connections:
- new net A5V: C14.1, C16.1, C20.1, C43.1, C47.1, C8.1, C9.1, IC1.8, IC2.8, IC4.8, U1.20, U11.6
- new net F: C6.1, C7.1, U1.22
- new net N$17: C21.1, R13.2
- new net N$20: C15.1, R12.2, R16.1, R17.1
- new net N$21: C23.1, IC2.2, R16.2
- new net N$23: C23.2, C24.1, IC2.1, R17.2
- new net N$24: C22.1, IC2.3, R14.2
- new net N$26: IC4.6, IC4.7
- new net N$29: C27.1, R21.2
- new net N$30: C25.1, R20.2, R23.1, R24.1
- new net N$31: C29.1, IC2.6, R23.2
- new net N$32: C29.2, C30.1, IC2.7, R24.2
- new net N$33: C28.1, IC2.5, R22.2
- new net N$58: C88.1, U11.4
- new net N$7: C12.1, IC1.6, R10.2
- new net N$8: C10.2, J-IN.T
- new net OUTA+: R11.1, U1.25
- new net OUTA-: R12.1, U1.24
- new net OUTB+: R19.1, U1.26
- new net OUTB-: R20.1, U1.27
- new net VQ1: C18.1, C19.1, IC4.3, IC4.5, U1.15
- new net VREF: C13.2, C4.2, IC4.1, IC4.2, R8.2, R9.2, U1.16, U1.19
- net +3V3: now also U1.10, U1.9; no longer U1.5, U1.8
- net +5V: now also C63.1, U11.1, U11.3; no longer C8.1, C9.1, U1.19
- net AGND: now also C14.2, C16.2, C18.2, C19.2, C20.2, C21.2, C22.2, C25.2, C26.2, C27.2, C28.2, C47.2, IC1.4, IC2.4, IC4.4, J-IN.S, J-IN.SW, J-OUT.S, J-OUT.SW, L3.1, R25.2, U1.21; no longer C11.2, C13.2, C4.2, C5.2, J1.1, J2.1, R10.2, R11.2, R13.2, R8.2, U1.20
- net GND: now also C43.2, C63.2, C88.2, L3.2, U1.2, U1.8, U11.2; no longer R18.1, U1.11, U1.12, U1.6
- net INA: now also C4.1, R5.1, R7.1, U1.17; no longer /INA.TP, C10.1, C11.1, U1.16
- net INB: now also R10.1, R6.1, U1.18; no longer /INB.TP, C12.1, U1.15
- net LRCK: now also U1.4; no longer /LRCK.TP, U1.2
- net MCLK: no longer /MCLK.TP
- net N$10: now also IC1.7, R6.2; no longer R10.1, R9.1
- net N$11: now also C5.2, J-IN.R; no longer J1.2, R7.2
- net N$12: now also C5.1, IC1.5, R9.1; no longer J1.3, R9.2
- net N$13: now also C24.2, R27.1; no longer C16.2, R13.1, R14.1
- net N$14: now also C30.2, R30.1; no longer C14.2, R11.1, R12.1
- net N$15: now also C26.1, R19.2, R21.1, R22.1; no longer C15.1, J2.2, R12.2
- net N$16: now also R11.2, R13.1, R14.1; no longer J2.3, R14.2
- net N$4: now also C11.1, IC1.2, R5.2; no longer C4.1, C5.1, U1.17
- net N$5: now also C11.2, IC1.1, R7.2; no longer C6.1, C7.1, U1.18
- net N$9: now also C10.1, IC1.3; no longer C10.2, R7.1
- net OUTA: now also J-OUT.T, R18.1, R27.2; no longer /OUTA.TP, C14.1, U1.23
- net OUTB: now also J-OUT.R, R25.1, R30.2; no longer /OUTB.TP, C16.1, U1.22
- net R-CODEC: no longer /RESET.TP
- net SCL: now also U1.11; no longer /SCL.TP, U1.10
- net SCLK: now also U1.5; no longer /SCLK.TP, U1.4
- net SDA: now also U1.12; no longer /SDA.TP, U1.9
- net SDIN: now also U1.7; no longer /SDIN.TP, U1.1
- net SDOUT: now also U1.6; no longer /SDOUT.TP, U1.7
Routing:
- net VREF: track 0.00 -> 81.3 mm, vias 0 -> 3
- net N$8: track 0.00 -> 32.3 mm, vias 0 -> 2
- net +3V3: track 93.3 -> 62.1 mm, vias 0 -> 1
- net OUTB+: track 0.00 -> 30.6 mm, vias 0 -> 2
- net OUTA+: track 0.00 -> 24.4 mm, vias 0 -> 2
- net OUTA-: track 0.00 -> 23.2 mm, vias 0 -> 2
- net SDIN: track 34.3 -> 11.2 mm, vias 2 -> 0
- net INA: track 9.11 -> 31.9 mm, vias 1 -> 0
- net R-CODEC: track 69.0 -> 46.9 mm
- net +5V: track 64.0 -> 44.3 mm
- net OUTB: track 10.7 -> 30.3 mm, vias 1 -> 0
- net INB: track 9.07 -> 26.2 mm, vias 1 -> 0
- net LRCK: track 25.2 -> 8.06 mm
- net OUTB-: track 0.00 -> 16.5 mm
- net VQ1: track 0.00 -> 16.2 mm
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- added copper zone on layer 16, net A5V
Other:
- board text added: "//////// norns/shield 211028"
- board text removed: "norns/shield 191106 monome.org"
